File: pcb_files/kicad_project/ZoroBot3.kicad_pcb (KiCad board)
At the start: 2 copper layers, 85.8 x 91.9 mm, 198 parts, among them Q1 NMOS, Q2 AON7423, Q3 ST-1KL3A, Q4 ST-1KL3A, Q5 ST-1KL3A, Q6 ST-1KL3A, U1 MPU-6500, U2 MPU-6500, Y1 Crystal_GND24

Commit message: Finaliza la version V1.2 con SRAM y correccion de errores.
Parts:
- removed AD8418AWBZ_1, AD8418AWBZ_2: ~, custom_footprints:SOP8
- removed C25, C27, C29, C36: 0.1uF, Capacitor_SMD:C_0402_1005Metric_Pad0.74x0.62mm_HandSolder
- removed C26: 0.01uF, Capacitor_SMD:C_0402_1005Metric_Pad0.74x0.62mm_HandSolder
- removed C28: 0.1uf, Capacitor_SMD:C_0402_1005Metric_Pad0.74x0.62mm_HandSolder
- removed DATA_MPU3: Conn_01x04_Socket, custom_footprints:ZoroBot3_Data_MPU
- removed JP3: Conn_01x01_Pin, custom_footprints:Generic_simple_1x_SMD_pin
- removed Q1: NMOS, Package_TO_SOT_SMD:SOT-23
- removed R12, R13: 0.05, Resistor_SMD:R_2512_6332Metric
- removed U1, U2: MPU-6500, Sensor_Motion:InvenSense_QFN-24_3x3mm_P0.4mm
- removed kibuzzard-6779A98A: G***, kibuzzard-6779A98A
- added CF1: 220nF, Capacitor_SMD:C_0402_1005Metric_Pad0.74x0.62mm_HandSolder, F.Cu at (141.8, 116.5)
- added CF2: 220nF, Capacitor_SMD:C_0402_1005Metric_Pad0.74x0.62mm_HandSolder, F.Cu at (161.6, 116.5)
- added CSRAM1: 0.1uF, Capacitor_SMD:C_0402_1005Metric_Pad0.74x0.62mm_HandSolder, F.Cu at (149.3, 110.1)
- added CSRAM2: 0.1uF, Capacitor_SMD:C_0402_1005Metric_Pad0.74x0.62mm_HandSolder, F.Cu at (114.3, 106.7)
- added DATA_MPU+SRAM1: Conn_01x05_Socket, custom_footprints:ZoroBot3_Data_MPU, F.Cu at (110.3, 98.3)
- added DS1: D, Diode_SMD:D_0805_2012Metric_Pad1.15x1.40mm_HandSolder, F.Cu at (125.9, 91.8)
- added LSM6DSR2: ~, Package_LGA:Bosch_LGA-14_3x2.5mm_P0.5mm, F.Cu at (110.3, 102.3)
- added MOSFET-N-SUC1: AO3400A, Package_TO_SOT_SMD:SOT-23, F.Cu at (120.3, 89.7)
- added RCM1: 5k, Resistor_SMD:R_0402_1005Metric_Pad0.72x0.64mm_HandSolder, F.Cu at (140.8, 115.6)
- added RCM2: 5k, Resistor_SMD:R_0402_1005Metric_Pad0.72x0.64mm_HandSolder, F.Cu at (139.6, 116.5)
- added RCM3: 5k, Resistor_SMD:R_0402_1005Metric_Pad0.72x0.64mm_HandSolder, F.Cu at (160.5, 115.6)
- added RCM4: 5k, Resistor_SMD:R_0402_1005Metric_Pad0.72x0.64mm_HandSolder, F.Cu at (159.4, 116.5)
- added RF1: 1k, Resistor_SMD:R_0402_1005Metric_Pad0.72x0.64mm_HandSolder, F.Cu at (140.8, 117.4)
- added RF2: 1k, Resistor_SMD:R_0402_1005Metric_Pad0.72x0.64mm_HandSolder, F.Cu at (160.5, 117.4)
- added RRAM1: 10K, Resistor_SMD:R_0402_1005Metric_Pad0.72x0.64mm_HandSolder, F.Cu at (152.0, 110.2)
- added RRAM2: 10K, Resistor_SMD:R_0402_1005Metric_Pad0.72x0.64mm_HandSolder, F.Cu at (114.3, 98.0)
- added SRAM1: 23AA04M-I/ST, Package_SO:TSSOP-8_4.4x3mm_P0.65mm, F.Cu at (150.7, 107.9)
- added SRAM2: 23AA04M-I/ST, Package_SO:TSSOP-8_4.4x3mm_P0.65mm, F.Cu at (114.3, 102.3)
- added kibuzzard-6A916D2B: G***, kibuzzard-6A916D2B, B.Cu at (126.7, 132.5)
- added kibuzzard-6A916D37: G***, kibuzzard-6A916D37, B.Cu at (126.7, 136.4)
- added kibuzzard-6A916D40: G***, kibuzzard-6A916D40, B.Cu at (126.7, 134.5)
- added kibuzzard-6A94423E: G***, kibuzzard-6A94423E, B.Cu at (190.3, 105.4)
- added kibuzzard-6A945D46: G***, kibuzzard-6A945D46, B.Cu at (150.6, 140.4)
- C39: value 0.01uF -> 0.1uF
- C43: value 10uF -> 47uF
- MOSFET-N1, MOSFET-N2, MOSFET-N3, MOSFET-N4: value AO3400 (A09T) -> AO3400A
- R18: value 200K -> 100K
- R19: value 47k -> 27k
- R24: value 100K -> 47K
- R25: value 10K -> 47K
- R26: value 20K -> 27K
- RS1, RS2, RS7, RS8: value 150 -> 33
- RS10, RS9: value 6.8K -> 1.5K
- RS3, RS4: value 6.8K -> 3.3K
- moved kibuzzard-6779A9B1 69.9 mm to (115.8, 105.8)
- moved R14 11.3 mm to (151.6, 97.1)
- moved R16 11.3 mm to (149.7, 97.1)
- moved R15 11.3 mm to (150.6, 97.1)
- moved C39 9.00 mm to (107.4, 101.2)
- moved C3 6.90 mm to (127.3, 84.4), turned to -83 degrees
- moved R10 4.99 mm to (166.1, 110.1)
- moved R7 4.99 mm to (163.2, 110.1)
- moved R8 4.99 mm to (164.2, 110.1)
- moved R6 4.99 mm to (162.3, 110.1)
- moved R9 4.99 mm to (165.1, 110.1)
- moved R3 4.95 mm to (137.0, 110.1)
- moved R5 4.95 mm to (138.9, 110.1)
- moved R2 4.95 mm to (136.1, 110.1)
- moved R4 4.95 mm to (138.0, 110.1)
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Connections:
- C37 pad 1: /Giroscopio/GND_MPU_B -> /Giroscopio/GND_MPU_A
- C37 pad 2: /Giroscopio/3.3_MPU_B -> /Giroscopio/3.3_MPU_A
- C38 pad 1: /Giroscopio/GND_MPU_B -> /Giroscopio/GND_MPU_A
- C38 pad 2: /Giroscopio/3.3_MPU_B -> /Giroscopio/3.3_MPU_A
- C39 pad 1: /Giroscopio/GND_MPU_A -> /Giroscopio/GND_MPU_B
- C39 pad 2: /Giroscopio/3.3_MPU_A -> /Giroscopio/3.3_MPU_B
- C40 pad 1: /Giroscopio/GND_MPU_A -> /Giroscopio/GND_MPU_B
- C40 pad 2: Net-(U2-REGOUT) -> /Giroscopio/3.3_MPU_B
- DATA_MPU2 pad 1: /Giroscopio/SPI_MISO_CONN_B -> /Giroscopio/SPI_MISO_CONN_A
- DATA_MPU2 pad 2: /Giroscopio/SPI_MOSI_CONN_B -> /Giroscopio/SPI_MOSI_CONN_A
- DATA_MPU2 pad 3: /Giroscopio/SPI_SCK_CONN_B -> /Giroscopio/SPI_SCK_CONN_A
- DATA_MPU2 pad 4: /Giroscopio/SPI_NSS_CONN_B -> /Giroscopio/SPI_NSS_CONN_A
- DEIXAME_QUE_PENSE_1 pad 33: unconnected-(DEIXAME_QUE_PENSE_1-PB12-Pad33) -> /NSS_SRAM
- LSM6DSR1 pad 1: /Giroscopio/SPI_MISO_CONN_B -> /Giroscopio/SPI_MISO_CONN_A
- LSM6DSR1 pad 12: /Giroscopio/SPI_NSS_CONN_B -> /Giroscopio/SPI_NSS_CONN_A
- LSM6DSR1 pad 13: /Giroscopio/SPI_SCK_CONN_B -> /Giroscopio/SPI_SCK_CONN_A
- LSM6DSR1 pad 14: /Giroscopio/SPI_MOSI_CONN_B -> /Giroscopio/SPI_MOSI_CONN_A
- LSM6DSR1 pad 2: Net-(JP3-Pin_1) -> /Giroscopio/3.3_MPU_A
- LSM6DSR1 pad 3: Net-(JP3-Pin_1) -> /Giroscopio/3.3_MPU_A
- LSM6DSR1 pad 5: /Giroscopio/3.3_MPU_B -> /Giroscopio/3.3_MPU_A
- LSM6DSR1 pad 6: /Giroscopio/GND_MPU_B -> /Giroscopio/GND_MPU_A
- LSM6DSR1 pad 7: /Giroscopio/GND_MPU_B -> /Giroscopio/GND_MPU_A
- LSM6DSR1 pad 8: /Giroscopio/3.3_MPU_B -> /Giroscopio/3.3_MPU_A
- MOSFET-N1 pad 1: Net-(LED_IR1-K) -> /Sensores/EMI_PA_D_CONN
- MOSFET-N1 pad 2: /Sensores/EMI_PA_D_CONN -> /Sensores/GND_D
- MOSFET-N1 pad 3: /Sensores/GND_D -> Net-(LED_IR1-K)
- MOSFET-N2 pad 1: Net-(LED_IR2-K) -> /Sensores/EMI_PA_I_CONN
- MOSFET-N2 pad 2: /Sensores/EMI_PA_I_CONN -> /Sensores/GND_I
- MOSFET-N2 pad 3: /Sensores/GND_I -> Net-(LED_IR2-K)
- MOSFET-N3 pad 1: Net-(LED_IR3-K) -> /Sensores/EMI_FRONT_D_CONN
- MOSFET-N3 pad 2: /Sensores/EMI_FRONT_D_CONN -> /Sensores/GND_FD
- MOSFET-N3 pad 3: /Sensores/GND_FD -> Net-(LED_IR3-K)
- MOSFET-N4 pad 1: Net-(LED_IR4-K) -> /Sensores/EMI_FRONT_I_CONN
- MOSFET-N4 pad 2: /Sensores/EMI_FRONT_I_CONN -> /Sensores/GND_FI
- MOSFET-N4 pad 3: /Sensores/GND_FI -> Net-(LED_IR4-K)
- PH1 pad 11: unconnected-(PH1-CM2-Pad11) -> /MOT_D_CM1
- PH1 pad 3: /SHUNT_MD -> /MOT_D+
- PH1 pad 7: unconnected-(PH1-CM1-Pad7) -> /MOT_D_CM1
- PH1 pad 8: /SHUNT_MD -> /MOT_D+
- PH2 pad 1: /SHUNT_MI -> /MOT_I-
- PH2 pad 10: /SHUNT_MI -> /MOT_I-
- PH2 pad 11: unconnected-(PH2-CM2-Pad11) -> /MOT_I_CM1
- PH2 pad 7: unconnected-(PH2-CM1-Pad7) -> /MOT_I_CM1
- POWER_MPU2 pad 1: /Giroscopio/GND_MPU_B -> /Giroscopio/GND_MPU_A
- POWER_MPU2 pad 2: /Giroscopio/3.3_MPU_B -> /Giroscopio/3.3_MPU_A
- POWER_MPU3 pad 1: /Giroscopio/GND_MPU_A -> /Giroscopio/GND_MPU_B
- POWER_MPU3 pad 2: /Giroscopio/3.3_MPU_A -> /Giroscopio/3.3_MPU_B
Routing:
- net +5V: track 164.6 -> 14.1 mm, vias 20 -> 12
- net /SHUNT_MI: track 63.9 -> 0.00 mm, vias 8 -> 0
- net /NSS_SRAM: track 0.00 -> 62.6 mm, vias 0 -> 3
- net /SHUNT_MD: track 51.0 -> 0.00 mm, vias 8 -> 0
- net /MOT_D+: track 20.6 -> 64.8 mm, vias 0 -> 8
- net +3V3: track 772.7 -> 809.9 mm, vias 33 -> 29
- net /MOT_I-: track 28.3 -> 63.2 mm, vias 0 -> 8
- net /Giroscopio/3.3_MPU_B: track 11.5 -> 39.7 mm, vias 3 -> 4
- net GND: track 198.4 -> 171.7 mm, vias 214 -> 302
- net /CURR_SEN_MI: track 56.8 -> 32.7 mm
- net /MOT_I_CM1: track 0.00 -> 23.9 mm, vias 0 -> 2
- net /MOT_D_CM1: track 0.00 -> 20.5 mm, vias 0 -> 2
- net /SEN_FRONT_I: track 99.5 -> 81.5 mm
- net /BATT: track 108.8 -> 125.4 mm, vias 37 -> 38
- net /CURR_SEN_MD: track 66.2 -> 50.2 mm
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- added copper zone on B.Cu, net /MOT_D+
- added copper zone on F.Cu, net /MOT_D+
- added copper zone on B.Cu, net /MOT_I-
- added copper zone on F.Cu, net /MOT_I-
- removed copper zone on B.Cu, net /SHUNT_MD
- removed copper zone on F.Cu, net /SHUNT_MD
- removed copper zone on B.Cu, net /SHUNT_MI
- removed copper zone on F.Cu, net /SHUNT_MI
Other:
- board size 85.8 x 91.9 mm -> 86.5 x 91.9 mm
- board text removed: "Component"
- board text removed: "Directly Below"
- board text removed: "JLCJLCJLCJLC"
- board text removed: "KEEPOUT"
- board text removed: "No Copper"
