File: pcb_files/kicad_project/ZoroBot3.kicad_sch (KiCad schematic)
At the start: 126 parts, among them Q1 NMOS, Q2 AON7423, U1 MPU-6500, Y1 Crystal_GND24

Commit message: Actualiza esquemático para añadir SRAM, lectura de corriente y diodo en succión
Parts:
- removed AD8418AWBZ_1, AD8418AWBZ_2: ~, custom_footprints:SOP8, symbol custom_symbols:AD8418
- removed C28: 0.1uf, Capacitor_SMD:C_0402_1005Metric_Pad0.74x0.62mm_HandSolder, symbol Device:C
- removed C29: 0.1uF, Capacitor_SMD:C_0402_1005Metric_Pad0.74x0.62mm_HandSolder, symbol Device:C
- removed R12, R13: 0.05, Resistor_SMD:R_2512_6332Metric, symbol Device:R
- added CF1, CF2: 220nF, Capacitor_SMD:C_0805_2012Metric, symbol Device:C
- added CSRAM1: 0.1uF, Capacitor_SMD:C_0402_1005Metric_Pad0.74x0.62mm_HandSolder, symbol Device:C
- added DS1: D, Diode_SMD:D_0805_2012Metric_Pad1.15x1.40mm_HandSolder, symbol Device:D
- added RCM1, RCM2, RCM3, RCM4: 5k, Resistor_SMD:R_0402_1005Metric_Pad0.72x0.64mm_HandSolder, symbol Device:R
- added RF1, RF2: 1k, Resistor_SMD:R_0402_1005Metric_Pad0.72x0.64mm_HandSolder, symbol Device:R
- added RRAM1: 10K, Resistor_SMD:R_0402_1005Metric_Pad0.72x0.64mm_HandSolder, symbol Device:R
- added SRAM1: 23AA04M-I/ST, Package_SO:TSSOP-8_4.4x3mm_P0.65mm, symbol custom_symbols:SRAM-23AA04M-I/ST
- BTN1, BTN2, BTN3, BTN_RST1, DC-DC1, IR_RECIVER1, MIC1, PH1, PH2, USB1: value ~ -> (none)
Connections:
- net SHUNT_MD is gone; now on net MOT_D+: PH1.3 (OUT2), PH1.8 (OUT2)
- net SHUNT_MI is gone; now on net MOT_I-: PH2.1 (OUT1), PH2.10 (OUT1)
- net +3V3: now also CSRAM1.2, RCM1.1, RCM3.1, RRAM1.2, SRAM1.3 (SIO2), SRAM1.7 (SIO3), SRAM1.8 (VCC)
- net BATT: now also DS1.1 (K)
- net CURR_SEN_MD: now also CF2.2, RF2.2
- net CURR_SEN_MI: now also CF1.2, RF1.2
- net GND: now also CF1.1, CF2.1, CSRAM1.1, RCM2.2, RCM4.2, SRAM1.4 (VSS)
- net MOT_S-: now also DS1.2 (A)
- net SPI_MISO: now also SRAM1.2 (SO/SIO1)
- net SPI_MOSI: now also SRAM1.5 (SI/SIO0)
- net SPI_SCK: now also SRAM1.6 (SCK)
- net MOT_I_CM1: now reaches PH2.11 (CM2)
- net MOT_I_CM1: now also PH2.7 (CM1), RCM1.2, RCM2.1, RF1.1
- net NSS_SRAM: now reaches DEIXAME_QUE_PENSE_1.33 (PB12)
- net NSS_SRAM: now also RRAM1.1, SRAM1.1 (CS)
- net MOT_D_CM1: now reaches PH1.11 (CM2)
- net MOT_D_CM1: now also PH1.7 (CM1), RCM3.2, RCM4.1, RF2.1
- no-connect marks 14 -> 9
Other:
- moved on the sheet: C23, C24, IR_RECIVER1, PH1, PH2, USB1

Commit message: Finaliza la version V1.2 con SRAM y correccion de errores.
Parts:
- removed C25, C27: 0.1uF, Capacitor_SMD:C_0402_1005Metric_Pad0.74x0.62mm_HandSolder, symbol Device:C
- removed C26: 0.01uF, Capacitor_SMD:C_0402_1005Metric_Pad0.74x0.62mm_HandSolder, symbol Device:C
- removed DATA_MPU1: Conn_01x04_Socket, custom_footprints:ZoroBot3_Data_MPU, symbol Connector:Conn_01x04_Socket
- removed POWER_MPU1: Conn_01x02_Socket, custom_footprints:ZoroBot3_Power_MPU, symbol Connector:Conn_01x02_Socket
- removed Q1: NMOS, Package_TO_SOT_SMD:SOT-23, symbol Simulation_SPICE:NMOS
- removed U1: MPU-6500, Sensor_Motion:InvenSense_QFN-24_3x3mm_P0.4mm, symbol PCB_ZoroBot_v3-rescue:MPU-6500-MPU-6500
- added MOSFET-N-SUC1: AO3400A, Package_TO_SOT_SMD:SOT-23, symbol Transistor_FET:AO3400A
- CF1, CF2: footprint Capacitor_SMD:C_0805_2012Metric -> Capacitor_SMD:C_0402_1005Metric_Pad0.74x0.62mm_HandSolder
Connections:
- net GND: now also MOSFET-N-SUC1.2 (S)
- net MOT_S-: now also MOSFET-N-SUC1.3 (D)
- net MOT_S_PWM: now also MOSFET-N-SUC1.1 (G)
- no-connect marks 9 -> 5
Other:
- note added: "MPU"
- note removed: "MPU-6500"
- note removed: "MPUs"
- moved on the sheet: BTN1, BTN2, BTN3, BTN_RST1, C23, C24, C30, C31, C44, C45, C46, C47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
